File: EuroClack_Formant_LFO_panel/EuroClack_Formant_LFO_panel.kicad_pcb (KiCad board)
At the start: 2 copper layers, 70.8 x 128.5 mm, 0 parts

Commit message: Added schematic pdf and made tweaks
Parts:
- added REF**: plated_rack_hole, BYOM_General:plated_rack_hole, F.Cu at (154.2, 40.9)
- added REF**: plated_rack_hole, BYOM_General:plated_rack_hole, F.Cu at (98.5, 41.0)
- added REF**: plated_rack_hole, BYOM_General:plated_rack_hole, F.Cu at (154.4, 163.5)
- added REF**: plated_rack_hole, BYOM_General:plated_rack_hole, F.Cu at (98.5, 163.5)
Other:
- outline, holes or cut-outs redrawn
